Commit message: update python

File: py/arx_x5_python/bimanual/script/x5.urdf (robot description, URDF)
Before this commit: robot ultron_v1.1_aa, 7 links, 6 joints
Links:
- link link6: mass 0.6000 -> 0.580

File: py/arx_x5_python/bimanual/script/x5_2025.urdf (robot description, URDF)
Before this commit: robot ultron_v1.1_aa, 7 links, 6 joints
Links:
- link link6: mass 0.650 -> 0.570
